File: Pendant PCB/Bottom_Board/Bottom.kicad_pcb (KiCad board)
At the start: 2 copper layers, 36 x 56 mm, 11 parts, among them J1 USB_B, J2 Conn_01x05, T1 Thumbstick_push

Commit message: Changes made for 2nd version.
Parts:
- D+1, D-1, GND1, VBUS1: footprint TestPoint:TestPoint_THTPad_2.0x2.0mm_Drill1.0mm -> TestPoint:TestPoint_THTPad_2.5x2.5mm_Drill1.2mm
- moved D-1 4.72 mm to (106.5, 110.5), turned to 180 degrees
- moved VBUS1 4.72 mm to (93.5, 110.5), turned to 180 degrees
- moved D+1 2.24 mm to (106.5, 115.0), turned to 180 degrees
- moved GND1 2.24 mm to (93.5, 115.0), turned to 180 degrees
Routing:
- net Net-(D-1-Pad1): track 52.5 -> 46.2 mm
- net Net-(J1-Pad1): track 53.3 -> 47.9 mm
- net Net-(D+1-Pad1): track 51.6 -> 54.0 mm
Other:
- outline, holes or cut-outs redrawn
