File: Pendant PCB/Bottom_Board/Bottom.sch (KiCad schematic (older format))
At the start: 11 parts, among them J1 USB_B, J2 Conn_01x05, T1 Thumbstick_push

Commit message: Boards finished and revised. Fabrication outputs generated.
Parts:
- renumbered TP2 to D+1, TP3 to D-1, TP4 to GND1, TP1 to VBUS1
Connections:
- net +5VA: now also T1.A2; no longer T1.C2
- net GND: now also GND1.1, J1.4 (GND), J2.3 (Pin_3), T1.C2; no longer J2.1 (Pin_1), T1.A2
- net at T1.B1: now also J2.1 (Pin_1); no longer J2.3 (Pin_3)
Other:
- moved on the sheet: J2
Changed lines of the file:
@@
 L Connector_Generic:Conn_01x05 J2
 U 1 1 5FF5C1AE
-P 4000 2450
-F 0 "J2" V 3964 2162 50  0000 R CNN
-F 1 "Conn_01x05" V 3873 2162 50  0000 R CNN
-F 2 "Connector_PinSocket_2.54mm:PinSocket_1x05_P2.54mm_Vertical" H 4000 2450 50  0001 C CNN
-F 3 "~" H 4000 2450 50  0001 C CNN
-	1    4000 2450
+P 4150 2450
+F 0 "J2" V 4114 2162 50  0000 R CNN
+F 1 "Conn_01x05" V 4023 2162 50  0000 R CNN
+F 2 "Connector_PinSocket_2.54mm:PinSocket_1x05_P2.54mm_Vertical" H 4150 2450 50  0001 C CNN
+F 3 "~" H 4150 2450 50  0001 C CNN
+	1    4150 2450
 	0    -1   -1   0
 $EndComp
@@
 	1    0    0    -1
 $EndComp
-$Comp
-L Connector:TestPoint TP1
-U 1 1 5FF60B59
-P 3900 5800
-F 0 "TP1" H 3958 5918 50  0000 L CNN
-F 1 "TestPoint" H 3958 5827 50  0000 L CNN
-F 2 "TestPoint:TestPoint_THTPad_2.0x2.0mm_Drill1.0mm" H 4100 5800 50  0001 C CNN
-F 3 "~" H 4100 5800 50  0001 C CNN
-	1    3900 5800
-	1    0    0    -1
-$EndComp
-$Comp
-L Connector:TestPoint TP2
-U 1 1 5FF60DBE
-P 4150 5700
-F 0 "TP2" H 4208 5818 50  0000 L CNN
-F 1 "TestPoint" H 4208 5727 50  0000 L CNN
-F 2 "TestPoint:TestPoint_THTPad_2.0x2.0mm_Drill1.0mm" H 4350 5700 50  0001 C CNN
-F 3 "~" H 4350 5700 50  0001 C CNN
-	1    4150 5700
-	1    0    0    -1
-$EndComp
-$Comp
-L Connector:TestPoint TP3
-U 1 1 5FF6100C
-P 4400 5600
-F 0 "TP3" H 4458 5718 50  0000 L CNN
-F 1 "TestPoint" H 4458 5627 50  0000 L CNN
-F 2 "TestPoint:TestPoint_THTPad_2.0x2.0mm_Drill1.0mm" H 4600 5600 50  0001 C CNN
-F 3 "~" H 4600 5600 50  0001 C CNN
-	1    4400 5600
-	1    0    0    -1
-$EndComp
-$Comp
-L Connector:TestPoint TP4
-U 1 1 5FF61213
-P 4650 5500
-F 0 "TP4" H 4708 5618 50  0000 L CNN
-F 1 "TestPoint" H 4708 5527 50  0000 L CNN
-F 2 "TestPoint:TestPoint_THTPad_2.0x2.0mm_Drill1.0mm" H 4850 5500 50  0001 C CNN
-F 3 "~" H 4850 5500 50  0001 C CNN
-	1    4650 5500
-	1    0    0    -1
-$EndComp
 Wire Wire Line
 	3700 5900 3900 5900
@@
 L power:GND #PWR0101
 U 1 1 5FF63686
-P 4250 4000
-F 0 "#PWR0101" H 4250 3750 50  0001 C CNN
-F 1 "GND" H 4255 3827 50  0000 C CNN
-F 2 "" H 4250 4000 50  0001 C CNN
-F 3 "" H 4250 4000 50  0001 C CNN
-	1    4250 4000
+P 4200 3950
+F 0 "#PWR0101" H 4200 3700 50  0001 C CNN
+F 1 "GND" H 4205 3777 50  0000 C CNN
+F 2 "" H 4200 3950 50  0001 C CNN
+F 3 "" H 4200 3950 50  0001 C CNN
+	1    4200 3950
 	1    0    0    -1
 $EndComp
@@
 Wire Wire Line
 	3650 3300 3750 3300
-Wire Wire Line
-	4250 4000 4250 3900
-Wire Wire Line
-	4150 3900 4250 3900
-Connection ~ 4250 3900
-Wire Wire Line
-	4250 3900 4250 3800
 $Comp
 L power:GND #PWR0103
 U 1 1 5FF66105
-P 3800 2750
-F 0 "#PWR0103" H 3800 2500 50  0001 C CNN
-F 1 "GND" H 3650 2700 50  0000 C CNN
-F 2 "" H 3800 2750 50  0001 C CNN
-F 3 "" H 3800 2750 50  0001 C CNN
-	1    3800 2750
+P 4150 2750
+F 0 "#PWR0103" H 4150 2500 50  0001 C CNN
+F 1 "GND" V 4150 2550 50  0000 C CNN
+F 2 "" H 4150 2750 50  0001 C CNN
+F 3 "" H 4150 2750 50  0001 C CNN
+	1    4150 2750
 	1    0    0    -1
 $EndComp
@@
 L power:+5VA #PWR0104
 U 1 1 5FF66493
-P 4250 3200
-F 0 "#PWR0104" H 4250 3050 50  0001 C CNN
-F 1 "+5VA" H 4265 3373 50  0000 C CNN
-F 2 "" H 4250 3200 50  0001 C CNN
-F 3 "" H 4250 3200 50  0001 C CNN
-	1    4250 3200
+P 4200 3250
+F 0 "#PWR0104" H 4200 3100 50  0001 C CNN
+F 1 "+5VA" H 4215 3423 50  0000 C CNN
+F 2 "" H 4200 3250 50  0001 C CNN
+F 3 "" H 4200 3250 50  0001 C CNN
+	1    4200 3250
 	1    0    0    -1
 $EndComp
@@
 L power:+5VA #PWR0105
 U 1 1 5FF67DB5
-P 3900 2750
-F 0 "#PWR0105" H 3900 2600 50  0001 C CNN
-F 1 "+5VA" H 3915 2923 50  0000 C CNN
-F 2 "" H 3900 2750 50  0001 C CNN
-F 3 "" H 3900 2750 50  0001 C CNN
-	1    3900 2750
+P 4050 2750
+F 0 "#PWR0105" H 4050 2600 50  0001 C CNN
+F 1 "+5VA" V 4050 2950 50  0000 C CNN
+F 2 "" H 4050 2750 50  0001 C CNN
+F 3 "" H 4050 2750 50  0001 C CNN
+	1    4050 2750
 	-1   0    0    1
 $EndComp
 Wire Wire Line
-	3800 2650 3800 2750
-Wire Wire Line
-	3900 2650 3900 2750
-Wire Wire Line
-	4250 3400 4250 3300
-Wire Wire Line
-	4150 3300 4250 3300
-Connection ~ 4250 3300
-Wire Wire Line
-	4250 3300 4250 3200
-Wire Wire Line
-	3950 3000 4000 3000
-Wire Wire Line
-	4000 3000 4000 2650
-Wire Wire Line
-	3950 3000 3950 3150
+	4150 2650 4150 2750
+Wire Wire Line
+	4050 2650 4050 2750
 Wire Wire Line
 	4400 3600 4450 3600
@@
 	4450 3600 4450 2950
 Wire Wire Line
-	4450 2950 4100 2950
-Wire Wire Line
-	4100 2950 4100 2650
-Wire Wire Line
 	3750 3900 3700 3900
 Wire Wire Line
@@
 Wire Wire Line
 	4550 4250 4550 2850
-Wire Wire Line
-	4550 2850 4200 2850
-Wire Wire Line
-	4200 2850 4200 2650
+$Comp
+L power:+5VA #PWR0106
+U 1 1 5FF661D2
+P 4300 3850
+F 0 "#PWR0106" H 4300 3700 50  0001 C CNN
+F 1 "+5VA" H 4315 4023 50  0000 C CNN
+F 2 "" H 4300 3850 50  0001 C CNN
+F 3 "" H 4300 3850 50  0001 C CNN
+	1    4300 3850
+	0    1    1    0
+$EndComp
+$Comp
+L power:GND #PWR0107
+U 1 1 5FF67607
+P 4300 3350
+F 0 "#PWR0107" H 4300 3100 50  0001 C CNN
+F 1 "GND" H 4305 3177 50  0000 C CNN
+F 2 "" H 4300 3350 50  0001 C CNN
+F 3 "" H 4300 3350 50  0001 C CNN
+	1    4300 3350
+	0    -1   -1   0
+$EndComp
+Wire Wire Line
+	4250 3400 4250 3350
+Wire Wire Line
+	4250 3350 4300 3350
+Wire Wire Line
+	4150 3300 4200 3300
+Wire Wire Line
+	4200 3300 4200 3250
+Wire Wire Line
+	4150 3900 4200 3900
+Wire Wire Line
+	4200 3900 4200 3950
+Wire Wire Line
+	4300 3850 4250 3850
+Wire Wire Line
+	4250 3850 4250 3800
+Wire Wire Line
+	3950 3150 3950 2650
+Wire Wire Line
+	4550 2850 4350 2850
+Wire Wire Line
+	4350 2850 4350 2650
+Wire Wire Line
+	4450 2950 4250 2950
+Wire Wire Line
+	4250 2950 4250 2650
+$Comp
+L power:GND #PWR0108
+U 1 1 5FF7C8BC
+P 3400 6600
+F 0 "#PWR0108" H 3400 6350 50  0001 C CNN
+F 1 "GND" H 3405 6427 50  0000 C CNN
+F 2 "" H 3400 6600 50  0001 C CNN
+F 3 "" H 3400 6600 50  0001 C CNN
+	1    3400 6600
+	1    0    0    -1
+$EndComp
+Wire Wire Line
+	3400 6600 3400 6550
+Connection ~ 3400 6550
+$Comp
+L Connector:TestPoint VBUS1
+U 1 1 5FF60B59
+P 3900 5800
+F 0 "VBUS1" H 3958 5918 50  0000 L CNN
+F 1 "TestPoint" H 3958 5827 50  0000 L CNN
+F 2 "TestPoint:TestPoint_THTPad_2.0x2.0mm_Drill1.0mm" H 4100 5800 50  0001 C CNN
+F 3 "~" H 4100 5800 50  0001 C CNN
+	1    3900 5800
+	1    0    0    -1
+$EndComp
+$Comp
+L Connector:TestPoint D+1
+U 1 1 5FF60DBE
+P 4150 5700
+F 0 "D+1" H 4208 5818 50  0000 L CNN
+F 1 "TestPoint" H 4208 5727 50  0000 L CNN
+F 2 "TestPoint:TestPoint_THTPad_2.0x2.0mm_Drill1.0mm" H 4350 5700 50  0001 C CNN
+F 3 "~" H 4350 5700 50  0001 C CNN
+	1    4150 5700
+	1    0    0    -1
+$EndComp
+$Comp
+L Connector:TestPoint D-1
+U 1 1 5FF6100C
+P 4400 5600
+F 0 "D-1" H 4458 5718 50  0000 L CNN
+F 1 "TestPoint" H 4458 5627 50  0000 L CNN
+F 2 "TestPoint:TestPoint_THTPad_2.0x2.0mm_Drill1.0mm" H 4600 5600 50  0001 C CNN
+F 3 "~" H 4600 5600 50  0001 C CNN
+	1    4400 5600
+	1    0    0    -1
+$EndComp
+$Comp
+L Connector:TestPoint GND1
+U 1 1 5FF61213
+P 4650 5500
+F 0 "GND1" H 4708 5618 50  0000 L CNN
+F 1 "TestPoint" H 4708 5527 50  0000 L CNN
+F 2 "TestPoint:TestPoint_THTPad_2.0x2.0mm_Drill1.0mm" H 4850 5500 50  0001 C CNN
+F 3 "~" H 4850 5500 50  0001 C CNN
+	1    4650 5500
+	1    0    0    -1
+$EndComp
 $EndSCHEMATC

Commit message: Changes made for 2nd version.
Parts:
- D+1, D-1, GND1, VBUS1: footprint TestPoint:TestPoint_THTPad_2.0x2.0mm_Drill1.0mm -> TestPoint:TestPoint_THTPad_2.5x2.5mm_Drill1.2mm
Changed lines of the file:
@@
 F 0 "VBUS1" H 3958 5918 50  0000 L CNN
 F 1 "TestPoint" H 3958 5827 50  0000 L CNN
-F 2 "TestPoint:TestPoint_THTPad_2.0x2.0mm_Drill1.0mm" H 4100 5800 50  0001 C CNN
+F 2 "TestPoint:TestPoint_THTPad_2.5x2.5mm_Drill1.2mm" H 4100 5800 50  0001 C CNN
 F 3 "~" H 4100 5800 50  0001 C CNN
 	1    3900 5800
@@
 F 0 "D+1" H 4208 5818 50  0000 L CNN
 F 1 "TestPoint" H 4208 5727 50  0000 L CNN
-F 2 "TestPoint:TestPoint_THTPad_2.0x2.0mm_Drill1.0mm" H 4350 5700 50  0001 C CNN
+F 2 "TestPoint:TestPoint_THTPad_2.5x2.5mm_Drill1.2mm" H 4350 5700 50  0001 C CNN
 F 3 "~" H 4350 5700 50  0001 C CNN
 	1    4150 5700
@@
 F 0 "D-1" H 4458 5718 50  0000 L CNN
 F 1 "TestPoint" H 4458 5627 50  0000 L CNN
-F 2 "TestPoint:TestPoint_THTPad_2.0x2.0mm_Drill1.0mm" H 4600 5600 50  0001 C CNN
+F 2 "TestPoint:TestPoint_THTPad_2.5x2.5mm_Drill1.2mm" H 4600 5600 50  0001 C CNN
 F 3 "~" H 4600 5600 50  0001 C CNN
 	1    4400 5600
@@
 F 0 "GND1" H 4708 5618 50  0000 L CNN
 F 1 "TestPoint" H 4708 5527 50  0000 L CNN
-F 2 "TestPoint:TestPoint_THTPad_2.0x2.0mm_Drill1.0mm" H 4850 5500 50  0001 C CNN
+F 2 "TestPoint:TestPoint_THTPad_2.5x2.5mm_Drill1.2mm" H 4850 5500 50  0001 C CNN
 F 3 "~" H 4850 5500 50  0001 C CNN
 	1    4650 5500
