File: Pendant PCB/Top_board/Pendant PCB.kicad_pcb (KiCad board)
At the start: 2 copper layers, 71 x 120.5 mm, 40 parts, among them J1 Conn_01x20, J2 Conn_01x20, J4 Conn_01x05, J5 Conn_02x02_Odd_Even

Commit message: Boards finished and revised. Fabrication outputs generated.
Parts:
- moved SW_$HX1 0.50 mm to (75.2, 106.8)
Connections:
- J4 pad 1: GND -> /A0
- J4 pad 3: /A0 -> GND
Routing:
- net /A0: track 116.8 -> 107.0 mm
- net /A2: track 127.6 -> 126.8 mm
Other:
- board size 71 x 120.5 mm -> 71 x 124 mm
