File: Pendant PCB/Top_board/Pendant PCB.sch (KiCad schematic (older format))
At the start: 40 parts, among them J1 Conn_01x20, J2 Conn_01x20, J4 Conn_01x05, J5 Conn_02x02_Odd_Even

Commit message: Boards finished and revised. Fabrication outputs generated.
Changed lines of the file:
@@
 L power:GND #PWR0136
 U 1 1 60033C28
-P 3600 2450
-F 0 "#PWR0136" H 3600 2200 50  0001 C CNN
-F 1 "GND" V 3605 2322 50  0000 R CNN
-F 2 "" H 3600 2450 50  0001 C CNN
-F 3 "" H 3600 2450 50  0001 C CNN
-	1    3600 2450
+P 3600 2250
+F 0 "#PWR0136" H 3600 2000 50  0001 C CNN
+F 1 "GND" V 3605 2122 50  0000 R CNN
+F 2 "" H 3600 2250 50  0001 C CNN
+F 3 "" H 3600 2250 50  0001 C CNN
+	1    3600 2250
 	0    -1   -1   0
 $EndComp
 Wire Wire Line
-	3250 2450 3600 2450
+	3250 2250 3600 2250
 Wire Wire Line
 	3250 2350 3600 2350
 Wire Wire Line
-	3250 2250 3600 2250
+	3250 2450 3600 2450
 Wire Wire Line
 	3250 2150 3600 2150
@@
 	0    1    1    0
 $EndComp
-Text Label 3350 2250 0    50   ~ 0
+Text Label 3350 2450 0    50   ~ 0
 J_X
 Text Label 3350 2150 0    50   ~ 0
